Commit message: mac version update

File: model/fr3.urdf (robot description, URDF)
Before this commit: robot panda, 12 links, 11 joints
Links:
- link panda_leftfinger: geometry collision mesh filename=finger_0.obj; visual mesh filename=finger_0.obj
- link panda_link1: geometry collision mesh filename=link1.stl; visual mesh filename=link1.obj
- link panda_link2: geometry collision mesh filename=link2.stl; visual mesh filename=link2.obj
- link panda_link3: geometry collision mesh filename=link3.stl; visual mesh filename=link3_0.obj
- link panda_link4: geometry collision mesh filename=link4.stl; visual mesh filename=link4_0.obj
- link panda_link5: geometry collision mesh filename=link5_collision_0.obj; collision mesh filename=link5_collision_1.obj
- link panda_link6: geometry collision mesh filename=link6.stl; visual mesh filename=link6_0.obj
- link panda_link7: geometry collision mesh filename=link7.stl; visual mesh filename=link7_0.obj
- link panda_rightfinger: geometry collision mesh filename=finger_0.obj; visual mesh filename=finger_0.obj
Joints:
- joint panda_joint1: limit lower=-2.7437 upper=2.7437 effort=87 velocity=2.62 -> lower=-2.9671 upper=2.9671 effort=87 velocity=2.1750
- joint panda_joint2: limit lower=-1.7837 upper=1.7837 effort=87 velocity=2.62 -> lower=-1.8326 upper=1.8326 effort=87 velocity=2.1750
- joint panda_joint3: limit lower=-2.9007 upper=2.9007 effort=87 velocity=2.62 -> lower=-2.9671 upper=2.9671 effort=87 velocity=2.1750
- joint panda_joint4: limit lower=-3.0421 upper=-0.1518 effort=87 velocity=2.62 -> lower=-3.1416 upper=0.0 effort=87 velocity=2.1750
- joint panda_joint5: limit lower=-2.8065 upper=2.8065 effort=12 velocity=5.2600 -> effort=12 velocity=2.6100
- joint panda_joint6: limit lower=0.5445 upper=4.5169 effort=12 velocity=4.18 -> lower=-0.0873 upper=3.8223 effort=12 velocity=2.6100
- joint panda_joint7: limit lower=-3.0159 upper=3.0159 effort=12 velocity=5.26 -> lower=-2.9671 upper=2.9671 effort=12 velocity=2.6100
